Commit message: saving manipulator progress

File: Environment/Divebot_Hybrid.urdf (robot description, URDF)
Before this commit: robot Divebot, 21 links, 20 joints
Links:
- link endEffector_left: geometry collision mesh filename=../../../model/ocean1/ocean1_graphics/HandO2_small.obj; visual mesh filename=../../../model/ocean1/ocean1_graphics/HandO2_small.obj
- link endEffector_right: geometry collision mesh filename=../../../model/ocean1/ocean1_graphics/HandO2_small.obj; visual mesh filename=../../../model/ocean1/ocean1_graphics/HandO2_small.obj
